File: Hardware/picoSense/docs/Schematic/picoPloT.kicad_sch (KiCad schematic)
At the start: 16 parts, among them J1 Debug, J2 Debug, J3 Temp, J4 Temp, J5 Conn_01x08_Pin, J6 Conn_01x08_Socket, SW1 RST, U1 MCU arm Cortex-M0x2, U10 MCP9808, U2 ePaper 2.13" Black/White (250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

Commit message: Move github account name to SloeComputers
Other:
- company: https://github.com/AnotherJohnH/picoPloT -> https://github.com/SloeComputers/picoPloT
Changed lines of the file:
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@@
     (date "2024-01-31")
     (rev "0.01")
-    (company "https://github.com/AnotherJohnH/picoPloT")
+    (company "https://github.com/SloeComputers/picoPloT")
   )
   (junction (at 222.25 95.25) (diameter 0) (color 0 0 0 0)
