File: Hardware/picoX21H/docs/Schematic/picoX21H.kicad_sch (KiCad schematic)
At the start: 21 parts, among them J1 Phones out, J2 Line out, J3 Debug, J4 Debug, J5 MIDI in, SW1 RST, U1 Pico 2 (RP2350), U2 Pico-Audio, U4 H11L1, U5 Waveshare 16x2 I2C LCD (AIP31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

Commit message: Move github account name to SloeComputers
Other:
- company: https://github.com/AnotherJohnH/picoX21H -> https://github.com/SloeComputers/picoX21H
Changed lines of the file:
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@@
     (date "2025-04-13")
     (rev "0.02")
-    (company "https://github.com/AnotherJohnH/picoX21H")
+    (company "https://github.com/SloeComputers/picoX21H")
   )
   (junction (at 271.78 52.07) (diameter 0) (color 0 0 0 0)
