File: Hardware/picoX7/docs/Schematics/picoX7.kicad_sch (KiCad schematic)
At the start: 42 parts, among them J1 MIDI in, J2 Debug, J3 Stereo line out, J4 Debug, J5 Stereo line out, J6 Stereo line out, SW1 RST, U1 Pico 2 (RP2350), U2 Pico-Audio, U3 H11L1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

Commit message: Move github account name to SloeComputers
Other:
- company: https://github.com/AnotherJohnH/picoX7 -> https://github.com/SloeComputers/picoX7
Changed lines of the file:
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@@
     (date "2024-10-01")
     (rev "0.05")
-    (company "https://github.com/AnotherJohnH/picoX7")
+    (company "https://github.com/SloeComputers/picoX7")
   )
   (junction (at 215.9 115.57) (diameter 0) (color 0 0 0 0)
