File: Hardware/picoX7/docs/Schematics/WAVESHARE_REV2_1/picoX7_WAVESHARE_REV2_1.kicad_sch (KiCad schematic)
At the start: 31 parts, among them J1 MIDI in, J2 Debug, J4 Debug, J5 Stereo line out, SW1 RST, U1 Pico 2 (RP2350), U3 H11L1, U4 74HCT164, U5 Waveshare 16x2 I2C LCD (AIP31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, U6 D1X8K-14BL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

Commit message: Move github account name to SloeComputers
Other:
- company: https://github.com/AnotherJohnH/picoX7 -> https://github.com/SloeComputers/picoX7
Changed lines of the file:
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@@
     (date "2024-10-01")
     (rev "0.06")
-    (company "https://github.com/AnotherJohnH/picoX7")
+    (company "https://github.com/SloeComputers/picoX7")
   )
   (junction (at 24.13 171.45) (diameter 0) (color 0 0 0 0)
